File: hardware/mainboard_PCB/kicad/sprig_console.kicad_sch (KiCad schematic)
At the start: 25 parts, among them J1 1020_battery_holder, J2 Conn_PinHeader_2x03_P2.54mm_V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, SW1 W, SW2 A, SW3 S, SW4 D, SW5 I, SW6 J, SW7 K, SW8 L, SW9 Slideswitch, U2 MAX98357AETE+, U5 Pico

Commit message: resdesign of KiCad board file to a fully through hole version
Parts:
- removed C2: 10uF, fab:C_1206, symbol fab:C
- removed C3: 0.1uF, fab:C_1206, symbol fab:C
- removed U1: ~, sprig:TFT_MSP1803, symbol sprig:TFT_MSP1803
- added R2: 100k, Resistor_THT:R_Axial_DIN0204_L3.6mm_D1.6mm_P5.08mm_Horizontal, symbol fab:R_1206
- added U1: Adafruit_TFT_ST7735, Library:Generic_1.8Inch_TFT_120x160, symbol fab_custom:Adafruit_TFT_ST7735
- C1, C4: footprint fab:C_1206 -> Capacitor_THT:C_Disc_D3.0mm_W1.6mm_P2.50mm; Silkscreen Value (none) -> 104
- D1, D2: footprint fab:LED_1206 -> PCM_4ms_LED:LED_3mm_C1A2_Polarity_Indicator
- D3: value SD1206T020S1R0 -> 1N5819; footprint fab:Diode_Schotky_100V_1A_Mini_SMA -> Diode_THT:D_DO-35_SOD27_P7.62mm_Horizontal
- J2: footprint fab:PinHeader_2x03_P2.54mm_Vertical_SMD -> Connector_PinHeader_2.54mm:PinHeader_2x03_P2.54mm_Vertical
- LS1: footprint fab:CVS-1508 -> Library:1W_8Ohm_Speaker
- R1, R3, R4: footprint fab:R_1206 -> Resistor_THT:R_Axial_DIN0204_L3.6mm_D1.6mm_P5.08mm_Horizontal
- SW9: footprint slideSWSMD:slideswitchCK -> Button_Switch_THT:SW_Slide-03_Wuerth-WS-SLTV_10x2.5x6.4_P2.54mm
- U2: footprint local:QFN50P300X300X80-17N -> Library:Max98357A_ClassD_I2S_Mono_Amp_BreakoutBoard
Connections:
- net +3V3: now also R2.1, U1.9 (VCC); no longer U2.8 (VDD)
- net BCLK: now also U2.2 (BCLK); no longer U2.16 (BCLK)
- net CARD_CS: now also U1.6 (CARD_CS)
- net DIN: now also U2.3 (DIN); no longer U2.1 (DIN)
- net D/C: now also U1.7 (D/C)
- net GND: now also U2.6 (GND), U1.10 (GND); no longer U2.11 (GND), U2.15 (GND), U2.2 (GAIN_SLOT), U2.3 (GND)
- net LITE: now also U1.1 (LITE)
- net LRCLK: now also U2.1 (LRC); no longer U2.14 (LRCLK)
- net MISO: now also U1.2 (MISO)
- net MOSI: now also U1.4 (MOSI)
- net RESET: now also U1.8 (RESET)
- net SCK: now also U1.3 (SCK)
- net TFT_CS: now also U1.5 (TFT_CS)
- net at LS1.1: now also U2.8 (-); no longer U2.10 (OUTN)
- net at U2.4 (GAIN): now also R2.2; no longer R1.2
- new net: R1.2, U2.5 (SD)
- no-connect marks 0 -> 7
Other:
- moved on the sheet: D2, R1, R4

Commit message: v1.1 board design complete for 38C3
Parts:
- C1, C4: footprint Capacitor_THT:C_Disc_D3.0mm_W1.6mm_P2.50mm -> Capacitor_THT:C_Disc_D4.3mm_W1.9mm_P5.00mm
- R1, R2, R3, R4: footprint Resistor_THT:R_Axial_DIN0204_L3.6mm_D1.6mm_P5.08mm_Horizontal -> Resistor_THT:R_Axial_DIN0204_L3.6mm_D1.6mm_P7.62mm_Horizontal
Changed lines of the file:
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@@
 			)
 		)
-		(property "Footprint" "Capacitor_THT:C_Disc_D3.0mm_W1.6mm_P2.50mm"
+		(property "Footprint" "Capacitor_THT:C_Disc_D4.3mm_W1.9mm_P5.00mm"
 			(at 164.7952 52.07 0)
 			(effects
@@
 			)
 		)
-		(property "Footprint" "Resistor_THT:R_Axial_DIN0204_L3.6mm_D1.6mm_P5.08mm_Horizontal"
+		(property "Footprint" "Resistor_THT:R_Axial_DIN0204_L3.6mm_D1.6mm_P7.62mm_Horizontal"
 			(at 114.3 124.46 90)
 			(effects
@@
 			)
 		)
-		(property "Footprint" "Resistor_THT:R_Axial_DIN0204_L3.6mm_D1.6mm_P5.08mm_Horizontal"
+		(property "Footprint" "Resistor_THT:R_Axial_DIN0204_L3.6mm_D1.6mm_P7.62mm_Horizontal"
 			(at 97.79 124.46 90)
 			(effects
@@
 			)
 		)
-		(property "Footprint" "Resistor_THT:R_Axial_DIN0204_L3.6mm_D1.6mm_P5.08mm_Horizontal"
+		(property "Footprint" "Resistor_THT:R_Axial_DIN0204_L3.6mm_D1.6mm_P7.62mm_Horizontal"
 			(at 134.62 121.92 90)
 			(effects
@@
 			)
 		)
-		(property "Footprint" "Resistor_THT:R_Axial_DIN0204_L3.6mm_D1.6mm_P5.08mm_Horizontal"
+		(property "Footprint" "Resistor_THT:R_Axial_DIN0204_L3.6mm_D1.6mm_P7.62mm_Horizontal"
 			(at 134.62 124.46 90)
 			(effects
@@
 			)
 		)
-		(property "Footprint" "Capacitor_THT:C_Disc_D3.0mm_W1.6mm_P2.50mm"
+		(property "Footprint" "Capacitor_THT:C_Disc_D4.3mm_W1.9mm_P5.00mm"
 			(at 82.2452 129.54 0)
 			(effects

Commit message: corrected capacitor silkscreening error, was 104 should be 105 for 1uf capacitor
Parts:
- C1, C4: Silkscreen Value 104 -> 105
Changed lines of the file:
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@@
 			)
 		)
-		(property "Silkscreen Value" "104"
+		(property "Silkscreen Value" "105"
 			(at 163.83 48.26 0)
 			(effects
@@
 			)
 		)
-		(property "Silkscreen Value" "104"
+		(property "Silkscreen Value" "105"
 			(at 81.28 125.73 0)
 			(effects
