File: hardware/mainboard_PCB/kicad/sprig_console.kicad_pcb (KiCad board)
At the start: 2 copper layers, 139.7 x 64.8 mm, 35 parts, among them J1 1020_battery_holder, J2 Conn_PinHeader_2x03_P2.54mm_V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, SW1 W, SW2 A, SW3 S, SW4 D, SW5 I, SW6 J, SW7 K, SW8 L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

Commit message: Created v1.4 for 39C3
Parts:
- added G***: LOGO, LOGO, B.Cu at (169.7, 120.4)
Other:
- board text added: "PCBS COURTESY OF:"
- board text added: "V1.4"
- board text added: "WayWayWay"
- board text removed: "AMAZE EDITION"
- board text removed: "JLCJLCJLCJLC"
- board text removed: "MADE AT:"
- board text removed: "V1.3"
